File: distribution_pcbs/y_carriage_board.brd (EAGLE design)
At the start: 60 x 65 mm, 11 parts

Commit message: change trace widths on y carriage board
Parts:
- LIMIT_OUT, ST_X_OUT, ST_Y_OUT, ST_Z_OUT: device SparkFun-Connectors:1X04 -> SparkFun-Connectors:MOLEX-1X4
Other:
- board size 60 x 65 mm -> 60 x 62.5 mm
Changed lines of the file:
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@@
 <plain>
 <wire x1="0" y1="0" x2="60" y2="0" width="0" layer="20"/>
-<wire x1="60" y1="0" x2="60" y2="65" width="0" layer="20"/>
-<wire x1="60" y1="65" x2="0" y2="65" width="0" layer="20"/>
-<wire x1="0" y1="65" x2="0" y2="0" width="0" layer="20"/>
+<wire x1="60" y1="0" x2="60" y2="62.5" width="0" layer="20"/>
+<wire x1="60" y1="62.5" x2="0" y2="62.5" width="0" layer="20"/>
+<wire x1="0" y1="62.5" x2="0" y2="0" width="0" layer="20"/>
 <text x="24.25" y="50.5" size="6.5" layer="16" font="vector" rot="MR0">X</text>
 <text x="24.25" y="32.5" size="6.5" layer="16" font="vector" rot="MR0">Y</text>
@@
 <element name="LIMIT_Y2" library="SparkFun-Connectors" package="MOLEX-1X2" value="M02POLAR" x="12" y="35" rot="R270"/>
 <element name="ST_X_IN" library="SparkFun-Connectors" package="MOLEX-1X4" value="" x="30" y="57" rot="R270"/>
-<element name="ST_X_OUT" library="SparkFun-Connectors" package="1X04" value="" x="45" y="50" rot="R270"/>
+<element name="ST_X_OUT" library="SparkFun-Connectors" package="MOLEX-1X4" value="" x="45" y="50" rot="R270"/>
 <element name="ST_Y1_IN" library="SparkFun-Connectors" package="MOLEX-1X4" value="" x="30" y="44" rot="R270"/>
 <element name="ST_Y2_IN" library="SparkFun-Connectors" package="MOLEX-1X4" value="" x="30" y="31" rot="R270"/>
-<element name="ST_Y_OUT" library="SparkFun-Connectors" package="1X04" value="" x="45" y="38" rot="R270"/>
+<element name="ST_Y_OUT" library="SparkFun-Connectors" package="MOLEX-1X4" value="" x="45" y="38" rot="R270"/>
 <element name="ST_Z_IN" library="SparkFun-Connectors" package="MOLEX-1X4" value="" x="30" y="18" rot="R270"/>
-<element name="ST_Z_OUT" library="SparkFun-Connectors" package="1X04" value="" x="45" y="22" rot="R270"/>
-<element name="LIMIT_OUT" library="SparkFun-Connectors" package="1X04" value="" x="30" y="4"/>
+<element name="ST_Z_OUT" library="SparkFun-Connectors" package="MOLEX-1X4" value="" x="45" y="22" rot="R270"/>
+<element name="LIMIT_OUT" library="SparkFun-Connectors" package="MOLEX-1X4" value="" x="30" y="4"/>
 <element name="LIMIT_IN" library="SparkFun-Connectors" package="MOLEX-1X4" value="" x="12" y="40.75" rot="R90"/>
 </elements>
@@
 <contactref element="LIMIT_OUT" pad="1"/>
 <contactref element="LIMIT_IN" pad="1"/>
-<wire x1="12" y1="40.75" x2="12" y2="35" width="0.75" layer="16"/>
-<wire x1="13.75" y1="35" x2="12" y2="35" width="0.75" layer="16"/>
-<wire x1="14.25" y1="18.5" x2="14.25" y2="28" width="0.75" layer="16"/>
-<wire x1="14.25" y1="28" x2="14.25" y2="34.5" width="0.75" layer="16"/>
-<wire x1="14.25" y1="18.5" x2="28.75" y2="4" width="0.75" layer="16"/>
-<wire x1="28.75" y1="4" x2="30" y2="4" width="0.75" layer="16"/>
-<wire x1="14.25" y1="34.5" x2="13.75" y2="35" width="0.75" layer="16"/>
-<wire x1="12" y1="28" x2="14.25" y2="28" width="0.75" layer="16"/>
+<wire x1="12" y1="40.75" x2="12" y2="35" width="1" layer="16"/>
+<wire x1="13.75" y1="35" x2="12" y2="35" width="1" layer="16"/>
+<wire x1="14.25" y1="18.5" x2="14.25" y2="28" width="1" layer="16"/>
+<wire x1="14.25" y1="28" x2="14.25" y2="34.5" width="1" layer="16"/>
+<wire x1="14.25" y1="18.5" x2="28.75" y2="4" width="1" layer="16"/>
+<wire x1="28.75" y1="4" x2="30" y2="4" width="1" layer="16"/>
+<wire x1="14.25" y1="34.5" x2="13.75" y2="35" width="1" layer="16"/>
+<wire x1="12" y1="28" x2="14.25" y2="28" width="1" layer="16"/>
 </signal>
 <signal name="N$10">
 <contactref element="LIMIT_OUT" pad="4"/>
 <contactref element="LIMIT_IN" pad="4"/>
-<wire x1="12" y1="48.37" x2="14.63" y2="48.37" width="0.75" layer="16"/>
-<wire x1="29.25" y1="8.25" x2="36" y2="8.25" width="0.75" layer="16"/>
-<wire x1="36" y1="8.25" x2="37.62" y2="6.63" width="0.75" layer="16"/>
-<wire x1="37.62" y1="6.63" x2="37.62" y2="4" width="0.75" layer="16"/>
-<wire x1="29.25" y1="8.25" x2="18" y2="19.5" width="0.75" layer="16"/>
-<wire x1="18" y1="19.5" x2="18" y2="45" width="0.75" layer="16"/>
-<wire x1="18" y1="45" x2="14.63" y2="48.37" width="0.75" layer="16"/>
+<wire x1="12" y1="48.37" x2="14.63" y2="48.37" width="1" layer="16"/>
+<wire x1="29.25" y1="8.25" x2="36" y2="8.25" width="1" layer="16"/>
+<wire x1="36" y1="8.25" x2="37.62" y2="6.63" width="1" layer="16"/>
+<wire x1="37.62" y1="6.63" x2="37.62" y2="4" width="1" layer="16"/>
+<wire x1="29.25" y1="8.25" x2="18" y2="19.5" width="1" layer="16"/>
+<wire x1="18" y1="19.5" x2="18" y2="45" width="1" layer="16"/>
+<wire x1="18" y1="45" x2="14.63" y2="48.37" width="1" layer="16"/>
 </signal>
 <signal name="N$11">
@@
 <contactref element="LIMIT_Y2" pad="2"/>
 <contactref element="LIMIT_OUT" pad="3"/>
-<wire x1="12" y1="25.46" x2="12" y2="17.75" width="0.75" layer="16"/>
-<wire x1="12" y1="17.75" x2="28" y2="1.75" width="0.75" layer="16"/>
-<wire x1="28" y1="1.75" x2="33.75" y2="1.75" width="0.75" layer="16"/>
-<wire x1="33.75" y1="1.75" x2="35.08" y2="3.08" width="0.75" layer="16"/>
-<wire x1="35.08" y1="3.08" x2="35.08" y2="4" width="0.75" layer="16"/>
-<wire x1="12" y1="32.46" x2="9.5" y2="29.96" width="0.75" layer="16"/>
-<wire x1="9.5" y1="29.96" x2="9.5" y2="26.75" width="0.75" layer="16"/>
-<wire x1="9.5" y1="26.75" x2="10.79" y2="25.46" width="0.75" layer="16"/>
-<wire x1="10.79" y1="25.46" x2="12" y2="25.46" width="0.75" layer="16"/>
+<wire x1="12" y1="25.46" x2="12" y2="17.75" width="1" layer="16"/>
+<wire x1="12" y1="17.75" x2="28" y2="1.75" width="1" layer="16"/>
+<wire x1="28" y1="1.75" x2="33.75" y2="1.75" width="1" layer="16"/>
+<wire x1="33.75" y1="1.75" x2="35.08" y2="3.08" width="1" layer="16"/>
+<wire x1="35.08" y1="3.08" x2="35.08" y2="4" width="1" layer="16"/>
+<wire x1="12" y1="32.46" x2="9.5" y2="29.96" width="1" layer="16"/>
+<wire x1="9.5" y1="29.96" x2="9.5" y2="26.75" width="1" layer="16"/>
+<wire x1="9.5" y1="26.75" x2="10.79" y2="25.46" width="1" layer="16"/>
+<wire x1="10.79" y1="25.46" x2="12" y2="25.46" width="1" layer="16"/>
 </signal>
 <signal name="N$17">
 <contactref element="LIMIT_OUT" pad="2"/>
 <contactref element="LIMIT_IN" pad="2"/>
-<wire x1="28.5" y1="7" x2="31.75" y2="7" width="0.75" layer="16"/>
-<wire x1="31.75" y1="7" x2="32.54" y2="6.21" width="0.75" layer="16"/>
-<wire x1="32.54" y1="6.21" x2="32.54" y2="4" width="0.75" layer="16"/>
-<wire x1="28.5" y1="7" x2="16.25" y2="19.25" width="0.75" layer="16"/>
-<wire x1="16.25" y1="19.25" x2="16.25" y2="41.75" width="0.75" layer="16"/>
-<wire x1="16.25" y1="41.75" x2="14.71" y2="43.29" width="0.75" layer="16"/>
-<wire x1="14.71" y1="43.29" x2="12" y2="43.29" width="0.75" layer="16"/>
+<wire x1="16.25" y1="19" x2="16.25" y2="41.75" width="1" layer="16"/>
+<wire x1="16.25" y1="41.75" x2="14.71" y2="43.29" width="1" layer="16"/>
+<wire x1="14.71" y1="43.29" x2="12" y2="43.29" width="1" layer="16"/>
+<wire x1="16.25" y1="19" x2="28.75" y2="6.5" width="1" layer="16"/>
+<wire x1="28.75" y1="6.5" x2="31.75" y2="6.5" width="1" layer="16"/>
+<wire x1="31.75" y1="6.5" x2="32.54" y2="5.71" width="1" layer="16"/>
+<wire x1="32.54" y1="5.71" x2="32.54" y2="4" width="1" layer="16"/>
 </signal>
 <signal name="N$25">
