File: distribution_pcbs/y_carriage_board.sch (EAGLE design)
At the start: 11 parts

Commit message: change trace widths on y carriage board
Parts:
- LIMIT_OUT, ST_X_OUT, ST_Y_OUT, ST_Z_OUT: device SparkFun-Connectors:M04PTH -> SparkFun-Connectors:M04POLAR
Changed lines of the file:
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@@
 <?xml version="1.0" encoding="utf-8"?>
 <!DOCTYPE eagle SYSTEM "eagle.dtd">
-<eagle version="7.1.0">
+<eagle version="7.2.0">
 <drawing>
 <settings>
@@
 <part name="LIMIT_Y1" library="SparkFun-Connectors" deviceset="M02" device="POLAR" value="M02POLAR"/>
 <part name="LIMIT_Y2" library="SparkFun-Connectors" deviceset="M02" device="POLAR" value="M02POLAR"/>
-<part name="ST_X_OUT" library="SparkFun-Connectors" deviceset="M04" device="PTH"/>
-<part name="ST_Y_OUT" library="SparkFun-Connectors" deviceset="M04" device="PTH"/>
-<part name="ST_Z_OUT" library="SparkFun-Connectors" deviceset="M04" device="PTH"/>
+<part name="ST_X_OUT" library="SparkFun-Connectors" deviceset="M04" device="POLAR"/>
+<part name="ST_Y_OUT" library="SparkFun-Connectors" deviceset="M04" device="POLAR"/>
+<part name="ST_Z_OUT" library="SparkFun-Connectors" deviceset="M04" device="POLAR"/>
 <part name="GND2" library="supply1" deviceset="GNDA" device=""/>
-<part name="LIMIT_OUT" library="SparkFun-Connectors" deviceset="M04" device="PTH"/>
+<part name="LIMIT_OUT" library="SparkFun-Connectors" deviceset="M04" device="POLAR"/>
 <part name="GND4" library="supply1" deviceset="GNDA" device=""/>
 <part name="LIMIT_IN" library="SparkFun-Connectors" deviceset="M04" device="POLAR"/>
