File: g_plus_shield/v1/g_plus_shield_v1.brd (EAGLE design)
At the start: 101.6 x 76.2 mm, 22 parts, among them Q1 IRF840

Commit message: outstanding work
Parts:
- C2, C3, C4: value (none) -> 0.1u
- R1, R4, R5: value (none) -> 220
- R2: value (none) -> 1m
- R3: value (none) -> 10k
